File: pcb/Blitzortung AS3935.kicad_pcb (KiCad board)
At the start: 2 copper layers, 0 parts

Commit message: first attempt of layout - many many VIAs but still home-made manufacturing possible. you have to connect the SC_CS wire with a bridge on a virtual third layer. no warranty....
Parts:
- added BT1: CR2032, KHZ 20PCB-V, F.Cu at (141.7, 116.7)
- added C1: 100n, SM0805, F.Cu at (149.7, 94.0)
- added C10: 100n, SM0805, B.Cu at (134.6, 102.4)
- added C11: 1u, SM0805, F.Cu at (126.0, 124.0)
- added C12: 1u, SM0805, B.Cu at (167.2, 104.3)
- added C13: 470u, Elko_vert_DM12-5_RM5, F.Cu at (119.8, 90.3)
- added C14: 1u, SM0805, F.Cu at (150.7, 96.3)
- added C15: 100n, SM0805, B.Cu at (157.1, 85.2)
- added C16: 1u, SM0805, F.Cu at (149.7, 116.5)
- added C17: 100n, SM0805, B.Cu at (120.2, 86.8)
- added C18: 100n, SM0805, F.Cu at (150.7, 98.5)
- added C19: 1u, SM0805, F.Cu at (155.7, 118.5)
- added C2: 100p, SM0805, F.Cu at (115.0, 116.0)
- added C20: 10n 50V, SM0805, B.Cu at (170.6, 93.8)
- added C21: 1u, SM0805, B.Cu at (186.5, 91.0)
- added C22: 47u Tantal, TantalC_SizeD_EIA-7343_HandSoldering_RevA_28Aug2012, B.Cu at (182.7, 103.6)
- added C23: 22p, SM0805, F.Cu at (148.7, 119.4)
- added C24: 22p, SM0805, F.Cu at (152.8, 119.4)
- added C25: 1u, SM0805, B.Cu at (116.6, 98.3)
- added C26: 1u, SM0805, B.Cu at (125.7, 104.2)
- added C27: 47u Tantal, TantalC_SizeD_EIA-7343_HandSoldering_RevA_28Aug2012, B.Cu at (136.8, 96.7)
- added C3: 100n, SM0805, F.Cu at (145.2, 99.8)
- added C4: 1n, SM0805, F.Cu at (117.0, 116.0)
- added C5: 10u, SM0805, F.Cu at (175.2, 92.8)
- added C6: 1u, SM0805, F.Cu at (173.0, 92.8)
- added C7: 10u, SM0805, F.Cu at (120.0, 110.0)
- added C8: 100n, SM0805, F.Cu at (142.9, 102.4)
- added C9: 1u, SM0805, F.Cu at (128.0, 122.0)
- added D1: p6ke39aSMD, Diode-SMB_Handsoldering_RevA_27July2010, B.Cu at (142.9, 85.0)
- added D2: SB150, Diode_DO-41_SOD81_Horizontal_RM10, B.Cu at (127.8, 86.9)
- added D3: PMEG6030, Diode-SMB_Handsoldering_RevA_27July2010, B.Cu at (167.2, 86.1)
- added D5: p6ke6,8aSMD, Diode-SMB_Handsoldering_RevA_27July2010, B.Cu at (160.1, 90.1)
- added D6: LED, LED-0805, F.Cu at (158.7, 112.1)
- added D7: 1n4148, Diode-MiniMELF_Handsoldering_RevA_27July2010, B.Cu at (119.8, 97.5)
- added D8: zf3,6SMD, Diode-MiniMELF_Handsoldering_RevA_27July2010, B.Cu at (122.7, 103.1)
- added D9: BPW34, GS2, F.Cu at (153.6, 93.9)
- added F1: MT 1A, FUSE5-20, F.Cu at (143.0, 87.0)
- added GS1: GS3, GS3, F.Cu at (132.0, 120.8)
- added HR1: DM3D-SF, DM3D-SF, F.Cu at (179.3, 94.0)
- added IC1: DS1307, SOIC-8_N, B.Cu at (161.8, 103.0)
- added IC2: ATMEGA328P-A, TQFP32, F.Cu at (150.6, 107.6)
- added K1: CONN_3_DHT, GS3, F.Cu at (162.4, 114.8)
- added L1: MA-5532, MA5532-AE, F.Cu at (112.0, 116.2)
- added L2: ferrit, SM0805, F.Cu at (155.1, 96.3)
- added L3: 68uH, Choke_SMD_Wuerth-WE-PD-Typ-LS_Handsoldering_RevA_27July2010, B.Cu at (178.7, 91.4)
- added LM1: LM2675, SO8N, B.Cu at (166.7, 93.8)
- added P1: CONN_2_pwr, PIN_ARRAY_2X1, F.Cu at (122.6, 82.1)
- added P10: CONN_1, 1pin, F.Cu at (112.5, 127.5)
- added P2: CONN_4_GPS, PIN_ARRAY_4x1, F.Cu at (135.9, 126.1)
- added P4: CONN_4_I2C, PIN_ARRAY_4x1, F.Cu at (122.5, 128.0)
- added P5: CONN_3X2_ISP, pin_array_3x2, F.Cu at (185.1, 115.7)
- added P6: CONN_6X2_ENC, pin_array_6x2, F.Cu at (169.2, 123.2)
- added P7: CONN_1, 1pin, F.Cu at (112.5, 82.5)
- added P8: CONN_1, 1pin, F.Cu at (187.5, 82.5)
- added P9: CONN_1, 1pin, F.Cu at (187.5, 127.5)
- added Q1: IRLML6401, SOT23GDS, F.Cu at (165.4, 102.9)
- added Q2: IRLML6401, SOT23GDS, F.Cu at (174.1, 118.0)
- added Q3: IRLML6401, SOT23GDS, F.Cu at (159.4, 121.1)
- added R10: 10k, SM0805, B.Cu at (125.4, 107.9)
- added R11: 10k, SM0805, B.Cu at (127.4, 109.8)
- added R12: 220, SM0805, F.Cu at (137.2, 110.6)
- added R13: 220, SM0805, F.Cu at (134.6, 110.6)
- added R15: 220, SM0805, F.Cu at (158.1, 115.5)
- added R16: 10k, SM0805, F.Cu at (158.5, 118.2)
- added R17: 0, MuSelf, B.Cu at (186.6, 108.9)
- added R18: 10k, SM0805, F.Cu at (177.1, 118.0)
- added R19: 200, SM0805, B.Cu at (118.5, 103.8)
- added R20: 330, SM0805, B.Cu at (118.5, 106.3)
- added R21: 10k, SM0805, F.Cu at (162.3, 118.2)
- added R3: 330k, SM0805, F.Cu at (144.6, 97.7)
- added R4: 10k, SM0805, F.Cu at (145.1, 102.4)
- added R5: 10k, SM0805, F.Cu at (119.0, 116.0)
- added R6: 39k, SM0805, F.Cu at (138.6, 102.4)
- added R7: 10k, SM0805, F.Cu at (140.8, 102.4)
- added R8: 22k, SM0805, B.Cu at (130.9, 100.2)
- added R9: 10k, SM0805, B.Cu at (134.6, 100.2)
- added U1: 74VHC125, SSOP-14, F.Cu at (170.3, 100.1)
- added U2: AS3935, QFN-16-P, F.Cu at (124.5, 115.5)
- added U3: LM317AT, TO220_VERT_123, F.Cu at (113.1, 100.2)
- added X1: Uhrenquarz, GS2, B.Cu at (166.9, 101.2)
- added X2: 20MHz, Crystal_HC49-SD_SMD_RevA_09Aug2010, F.Cu at (150.5, 124.2)
Routing:
- net GND: track 0.00 -> 329.0 mm, vias 0 -> 11
- net +5V: track 0.00 -> 319.2 mm, vias 0 -> 11
- net GNDPWR: track 0.00 -> 125.4 mm
- net +3.3V: track 0.00 -> 123.1 mm, vias 0 -> 4
- net /eth_so: track 0.00 -> 76.0 mm, vias 0 -> 3
- net /scl: track 0.00 -> 74.4 mm, vias 0 -> 2
- net /eth_sck: track 0.00 -> 72.3 mm, vias 0 -> 1
- net Net-(C13-Pad1): track 0.00 -> 71.5 mm, vias 0 -> 2
- net /eth_si: track 0.00 -> 67.7 mm, vias 0 -> 2
- net /IRQ_SD: track 0.00 -> 66.0 mm, vias 0 -> 2
- net /sda: track 0.00 -> 65.7 mm, vias 0 -> 2
- net VCC: track 0.00 -> 50.1 mm, vias 0 -> 2
- net /eth_cs: track 0.00 -> 47.4 mm, vias 0 -> 1
- net /reset: track 0.00 -> 45.9 mm, vias 0 -> 3
- net Net-(BT1-Pad1): track 0.00 -> 39.5 mm
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- added copper zone on B.Cu, net GND
- added copper zone on F.Cu, net GND
- added copper zone on B.Cu, net GNDPWR
- added copper zone on F.Cu, net GNDPWR
Other:
- board outline added: 80 x 50 mm
- net class Default: clearance 0.254 -> 0.2032; via_dia 0.889 -> 1.5; via_drill 0.635 -> 0.9
- rule trace_clearance: 0.254 -> 0.2032
- rule trace_min: 0.254 -> 0.2032
- board text added: "ACHTUNG ENTWICKLUNGSMUSTER: 1. Uhrenquarz muss an Lötpads gelötet werden 2. SD_CS muss mit einem Stück Draht verbunden werden 16.11.2013 - PhilippH"
- board text added: "Blitz- sucher"
- board text added: "Fläche für PowerGND"
- board text added: "keine Fläche!"
